Commit message: update mf_localization and configuration files to keep compatibility with the TF tree of cabot-description
- change the default value of published_frame from base_link to base_control_shift to keep the compatibility with the TF tree of cabot-description
- update simplified urdf files in mf_localization_mapping define use base_control_shift

Signed-off-by: Masayuki Murata <muratams@jp.ibm.com>

File: mf_localization_mapping/urdf/cabot2-e2.urdf (robot description, URDF)
Before this commit: robot cabot2-e2, 7 links, 6 joints
Links:
- added link base_control_shift
Joints:
- added joint control_center_joint: type fixed, parent base_control_shift, child base_link, origin xyz=0.0 0.0 0.0 rpy=0.0 0.0 0.0

File: mf_localization_mapping/urdf/cabot2-gt1.urdf (robot description, URDF)
Before this commit: robot cabot2-gt1, 7 links, 6 joints
Links:
- added link base_control_shift
Joints:
- added joint control_center_joint: type fixed, parent base_control_shift, child base_link, origin xyz=0.0 0.0 0.0 rpy=0.0 0.0 0.0

File: mf_localization_mapping/urdf/cabot2-gtm-outdoor.urdf (robot description, URDF)
Before this commit: robot cabot2-gtm, 7 links, 6 joints
Links:
- added link base_control_shift
Joints:
- added joint control_center_joint: type fixed, parent base_control_shift, child base_link, origin xyz=0.0 0.0 0.0 rpy=0.0 0.0 0.0

File: mf_localization_mapping/urdf/rover.urdf (robot description, URDF)
Before this commit: robot rover, 5 links, 4 joints
Links:
- added link base_control_shift
Joints:
- added joint control_center_joint: type fixed, parent base_control_shift, child base_link, origin xyz=0.0 0.0 0.0 rpy=0.0 0.0 0.0

File: mf_localization_mapping/urdf/tripod.urdf (robot description, URDF)
Before this commit: robot tripod, 5 links, 4 joints
Links:
- added link base_control_shift
Joints:
- added joint control_center_joint: type fixed, parent base_control_shift, child base_link, origin xyz=0.0 0.0 0.0 rpy=0.0 0.0 0.0
